File: HW/CNC/PB_Panel/PB_Panel.kicad_pcb (KiCad board)
At the start: 2 copper layers, 109.2 x 50.8 mm, 19 parts, among them J1 1x11 2.54mm female 90deg, SW1 RED, SW10 RED, SW11 BLUE, SW12 BLUE, SW13 YELLOW, SW14 YELLOW, SW15 GRAY, SW16 GRAY, SW17 BLACK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

Commit message: Finished PCB.
Parts:
- added H1: Board leg mounting hole, MountingHole:MountingHole_3.2mm_M3, F.Cu at (2.54, 27.9)
- added H2: Board leg mounting hole, MountingHole:MountingHole_3.2mm_M3, F.Cu at (2.54, 38.1)
- J1: value 1x11 2.54mm female 90deg -> 1x9 2.54mm female 90deg; footprint Connector_PinSocket_2.54mm:PinSocket_1x11_P2.54mm_Horizontal -> Connector_PinSocket_2.54mm:PinSocket_1x09_P2.54mm_Horizontal
- moved J1 235.3 mm to (-50.8, 5.08), turned to 0 degrees
- moved SW3 5.12 mm to (-33.0, 17.8), turned to -90 degrees
Connections:
- J1 pad 1: GND -> /N_R3
- J1 pad 2: VCC -> /N_R0
- J1 pad 3: /N_C0 -> /N_C2
- J1 pad 4: /N_C1 -> /N_C3
- J1 pad 5: /N_C2 -> /N_C4
- J1 pad 6: /N_C3 -> /N_C0
- J1 pad 7: /N_C4 -> /N_R1
- J1 pad 8: /N_C5 -> /N_R2
- J1 pad 9: /N_R0 -> /N_C1
- SW1 pad 1: unconnected-(SW1-Pad1) -> /N_C1
- SW1 pad 2: unconnected-(SW1-Pad2) -> /N_R2
- SW10 pad 1: unconnected-(SW10-Pad1) -> /N_C3
- SW10 pad 2: unconnected-(SW10-Pad2) -> /N_R2
- SW11 pad 1: unconnected-(SW11-Pad1) -> /N_C4
- SW11 pad 2: unconnected-(SW11-Pad2) -> /N_R0
- SW12 pad 1: unconnected-(SW12-Pad1) -> /N_C4
- SW12 pad 2: unconnected-(SW12-Pad2) -> /N_R2
- SW13 pad 1: unconnected-(SW13-Pad1) -> /N_C2
- SW13 pad 2: unconnected-(SW13-Pad2) -> /N_R1
- SW14 pad 1: unconnected-(SW14-Pad1) -> /N_C2
- SW14 pad 2: unconnected-(SW14-Pad2) -> /N_R3
- SW15 pad 1: unconnected-(SW15-Pad1) -> /N_C3
- SW15 pad 2: unconnected-(SW15-Pad2) -> /N_R1
- SW16 pad 1: unconnected-(SW16-Pad1) -> /N_C3
- SW16 pad 2: unconnected-(SW16-Pad2) -> /N_R3
- SW17 pad 1: unconnected-(SW17-Pad1) -> /N_C4
- SW17 pad 2: unconnected-(SW17-Pad2) -> /N_R1
- SW18 pad 1: unconnected-(SW18-Pad1) -> /N_C4
- SW18 pad 2: unconnected-(SW18-Pad2) -> /N_R3
- SW2 pad 1: unconnected-(SW2-Pad1) -> /N_C0
- SW2 pad 2: unconnected-(SW2-Pad2) -> /N_R2
- SW3 pad 1: unconnected-(SW3-Pad1) -> /N_C0
- SW3 pad 2: unconnected-(SW3-Pad2) -> /N_R1
- SW4 pad 1: unconnected-(SW4-Pad1) -> /N_C0
- SW4 pad 2: unconnected-(SW4-Pad2) -> /N_R3
- SW5 pad 1: unconnected-(SW5-Pad1) -> /N_C1
- SW5 pad 2: unconnected-(SW5-Pad2) -> /N_R1
- SW6 pad 1: unconnected-(SW6-Pad1) -> /N_C1
- SW6 pad 2: unconnected-(SW6-Pad2) -> /N_R3
- SW7 pad 1: unconnected-(SW7-Pad1) -> /N_C2
- SW7 pad 2: unconnected-(SW7-Pad2) -> /N_R0
- SW8 pad 1: unconnected-(SW8-Pad1) -> /N_C2
- SW8 pad 2: unconnected-(SW8-Pad2) -> /N_R2
- SW9 pad 1: unconnected-(SW9-Pad1) -> /N_C3
- SW9 pad 2: unconnected-(SW9-Pad2) -> /N_R0
Routing:
- net /N_R3: track 0.00 -> 193.0 mm, vias 0 -> 2
- net /N_R2: track 0.00 -> 130.2 mm, vias 0 -> 2
- net /N_C3: track 0.00 -> 129.6 mm, vias 0 -> 2
- net /N_R1: track 0.00 -> 116.9 mm
- net /N_C4: track 0.00 -> 116.8 mm
- net /N_C2: track 0.00 -> 114.4 mm, vias 0 -> 4
- net /N_R0: track 0.00 -> 111.7 mm
- net /N_C0: track 0.00 -> 99.0 mm, vias 0 -> 2
- net /N_C1: track 0.00 -> 73.7 mm, vias 0 -> 2
Other:
- board size 109.2 x 50.8 mm -> 106.7 x 48.3 mm
