File: HW/CNC/CNC_Panel_Harness/CNC_Panel_Harness.kicad_sch (KiCad schematic)
At the start: 3 parts, among them J1 1x8 2.54mm male 90deg, J2 1x9 2.54mm male 90deg

Commit message: Correction
Parts:
- J2: Comment (none) -> To PB_Panel
Changed lines of the file:
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@@
       (effects (font (size 1.27 1.27)) hide)
     )
+    (property "Comment" "To PB_Panel" (id 4) (at 191.77 79.375 0))
     (pin "1")
     (pin "2")
